File: board/untitled.brd (EAGLE design)
At the start: 100 x 80 mm, 32 parts, among them IC1 PIC16F628P, IC2 LP2950CZ-3.3, Q1 BC546B, Q2 BC546B

Commit message: WIP test in isolation
Parts:
- R1, R10, R12, R2, R4, R5, R8: value (none) -> 47k
- R11, R13: value (none) -> 10k
- R3, R6, R7, R9: value (none) -> 100k
Connections:
- removed net +12V: C1.1, C4.1, IC2.3, TP8.TP
- net +5V: now also C1.1, C4.1, IC2.3, TP8.TP
Routing:
- net GND: track 0.00 -> 125.2 mm
- net +3V3: track 0.00 -> 92.5 mm
- net +5V: track 0.00 -> 53.2 mm
- net N$21: track 0.00 -> 38.5 mm
- net N$7: track 0.00 -> 36.6 mm
- net N$3: track 0.00 -> 35.2 mm
- net N$5: track 0.00 -> 35.1 mm
- net N$2: track 0.00 -> 34.4 mm
- net N$4: track 0.00 -> 30.8 mm
- net N$1: track 0.00 -> 26.6 mm
- net N$16: track 0.00 -> 17.6 mm
- net N$13: track 0.00 -> 11.6 mm
- net N$19: track 0.00 -> 11.0 mm
- net N$22: track 0.00 -> 6.35 mm
- net N$12: track 0.00 -> 6.26 mm
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
Commit message: - Added notes
Parts:
- renumbered TP2 to CE, TP3 to CLK, TP4 to DAT, TP5 to MONO, TP6 to TUNE, TP7 to STEREO
Changed lines of the file:
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@@
 </element>
 <element name="R10" library="rcl" library_urn="urn:adsk.eagle:library:334" package="0204/7" package3d_urn="urn:adsk.eagle:package:23498/2" value="47k" x="39.37" y="33.02" smashed="yes" rot="R270">
-<attribute name="NAME" x="40.5384" y="35.1536" size="1.27" layer="25" ratio="10" rot="R270"/>
+<attribute name="NAME" x="39.2684" y="35.1536" size="1.27" layer="25" ratio="10" rot="R270"/>
 <attribute name="POPULARITY" value="79" x="0" y="-2.54" size="1.778" layer="27" rot="R270" display="off"/>
 <attribute name="SPICEPREFIX" value="R" x="0" y="-2.54" size="1.778" layer="27" rot="R270" display="off"/>
@@
 </element>
 <element name="TP1" library="testpad" library_urn="urn:adsk.eagle:library:385" package="B1,27" package3d_urn="urn:adsk.eagle:package:27944/2" value="TPB1,27" x="39.37" y="26.67" smashed="yes">
-<attribute name="NAME" x="38.735" y="27.686" size="1.27" layer="25" ratio="10"/>
+<attribute name="NAME" x="20.955" y="27.686" size="1.27" layer="25" ratio="10"/>
 <attribute name="POPULARITY" value="19" x="60.96" y="-7.62" size="1.778" layer="27" display="off"/>
 <attribute name="TP_SIGNAL_NAME" value="" x="38.735" y="24.765" size="1" layer="37"/>
 <attribute name="VALUE" x="38.735" y="24.638" size="0.0254" layer="27"/>
 </element>
-<element name="TP2" library="testpad" library_urn="urn:adsk.eagle:library:385" package="B1,27" package3d_urn="urn:adsk.eagle:package:27944/2" value="TPB1,27" x="54.61" y="21.59" smashed="yes">
-<attribute name="NAME" x="53.975" y="22.606" size="1.27" layer="25" ratio="10"/>
+<element name="CE" library="testpad" library_urn="urn:adsk.eagle:library:385" package="B1,27" package3d_urn="urn:adsk.eagle:package:27944/2" value="TPB1,27" x="54.61" y="21.59" smashed="yes">
+<attribute name="NAME" x="59.055" y="22.606" size="1.27" layer="25" ratio="10"/>
 <attribute name="POPULARITY" value="19" x="54.61" y="21.59" size="1.778" layer="27" display="off"/>
 <attribute name="TP_SIGNAL_NAME" value="" x="54.61" y="21.59" size="1.778" layer="27" display="off"/>
 <attribute name="VALUE" x="53.975" y="20.828" size="0.0254" layer="27"/>
 </element>
-<element name="TP3" library="testpad" library_urn="urn:adsk.eagle:library:385" package="B1,27" package3d_urn="urn:adsk.eagle:package:27944/2" value="TPB1,27" x="39.37" y="17.78" smashed="yes">
-<attribute name="NAME" x="34.925" y="17.526" size="1.27" layer="25" ratio="10"/>
+<element name="CLK" library="testpad" library_urn="urn:adsk.eagle:library:385" package="B1,27" package3d_urn="urn:adsk.eagle:package:27944/2" value="TPB1,27" x="39.37" y="17.78" smashed="yes">
+<attribute name="NAME" x="17.145" y="18.796" size="1.27" layer="25" ratio="10"/>
 <attribute name="POPULARITY" value="19" x="39.37" y="17.78" size="1.778" layer="27" display="off"/>
 <attribute name="TP_SIGNAL_NAME" value="" x="39.37" y="17.78" size="1.778" layer="27" display="off"/>
 <attribute name="VALUE" x="38.735" y="17.018" size="0.0254" layer="27"/>
 </element>
-<element name="TP4" library="testpad" library_urn="urn:adsk.eagle:library:385" package="B1,27" package3d_urn="urn:adsk.eagle:package:27944/2" value="TPB1,27" x="36.83" y="45.72" smashed="yes">
-<attribute name="NAME" x="38.735" y="45.466" size="1.27" layer="25" ratio="10"/>
+<element name="DAT" library="testpad" library_urn="urn:adsk.eagle:library:385" package="B1,27" package3d_urn="urn:adsk.eagle:package:27944/2" value="TPB1,27" x="36.83" y="45.72" smashed="yes">
+<attribute name="NAME" x="19.685" y="44.196" size="1.27" layer="25" ratio="10"/>
 <attribute name="POPULARITY" value="19" x="36.83" y="45.72" size="1.778" layer="27" display="off"/>
 <attribute name="TP_SIGNAL_NAME" value="" x="36.83" y="45.72" size="1.778" layer="27" display="off"/>
 <attribute name="VALUE" x="36.195" y="44.958" size="0.0254" layer="27"/>
 </element>
-<element name="TP5" library="testpad" library_urn="urn:adsk.eagle:library:385" package="B1,27" package3d_urn="urn:adsk.eagle:package:27944/2" value="TPB1,27" x="54.61" y="31.75" smashed="yes">
-<attribute name="NAME" x="53.975" y="32.766" size="1.27" layer="25" ratio="10"/>
+<element name="MONO" library="testpad" library_urn="urn:adsk.eagle:library:385" package="B1,27" package3d_urn="urn:adsk.eagle:package:27944/2" value="TPB1,27" x="54.61" y="31.75" smashed="yes">
+<attribute name="NAME" x="59.055" y="34.036" size="1.27" layer="25" ratio="10"/>
 <attribute name="POPULARITY" value="19" x="54.61" y="31.75" size="1.778" layer="27" display="off"/>
 <attribute name="TP_SIGNAL_NAME" value="" x="54.61" y="31.75" size="1.778" layer="27" display="off"/>
 <attribute name="VALUE" x="53.975" y="30.988" size="0.0254" layer="27"/>
 </element>
-<element name="TP6" library="testpad" library_urn="urn:adsk.eagle:library:385" package="B1,27" package3d_urn="urn:adsk.eagle:package:27944/2" value="TPB1,27" x="35.56" y="49.53" smashed="yes">
-<attribute name="NAME" x="34.925" y="50.546" size="1.27" layer="25" ratio="10"/>
+<element name="TUNE" library="testpad" library_urn="urn:adsk.eagle:library:385" package="B1,27" package3d_urn="urn:adsk.eagle:package:27944/2" value="TPB1,27" x="35.56" y="49.53" smashed="yes">
+<attribute name="NAME" x="31.115" y="50.546" size="1.27" layer="25" ratio="10"/>
 <attribute name="POPULARITY" value="19" x="35.56" y="49.53" size="1.778" layer="27" display="off"/>
 <attribute name="TP_SIGNAL_NAME" value="" x="35.56" y="49.53" size="1.778" layer="27" display="off"/>
 <attribute name="VALUE" x="34.925" y="48.768" size="0.0254" layer="27"/>
 </element>
-<element name="TP7" library="testpad" library_urn="urn:adsk.eagle:library:385" package="B1,27" package3d_urn="urn:adsk.eagle:package:27944/2" value="TPB1,27" x="45.72" y="52.07" smashed="yes">
-<attribute name="NAME" x="45.085" y="53.086" size="1.27" layer="25" ratio="10"/>
+<element name="STEREO" library="testpad" library_urn="urn:adsk.eagle:library:385" package="B1,27" package3d_urn="urn:adsk.eagle:package:27944/2" value="TPB1,27" x="45.72" y="52.07" smashed="yes">
+<attribute name="NAME" x="57.785" y="53.086" size="1.27" layer="25" ratio="10"/>
 <attribute name="POPULARITY" value="19" x="45.72" y="52.07" size="1.778" layer="27" display="off"/>
 <attribute name="TP_SIGNAL_NAME" value="" x="45.72" y="52.07" size="1.778" layer="27" display="off"/>
@@
 <wire x1="52.1208" y1="29.1084" x2="52.07" y2="29.21" width="0.1524" layer="1"/>
 <wire x1="41.91" y1="34.29" x2="36.83" y2="34.29" width="0.1524" layer="1"/>
-<wire x1="25.2984" y1="12.8016" x2="25.2984" y2="11.43" width="0.1524" layer="1"/>
+<wire x1="25.2984" y1="12.8016" x2="25.4" y2="11.3284" width="0.1524" layer="1"/>
 <wire x1="22.86" y1="15.24" x2="23.4696" y2="14.6304" width="0.1524" layer="1"/>
 <wire x1="23.4696" y1="14.6304" x2="25.2984" y2="12.8016" width="0.1524" layer="1"/>
-<wire x1="25.2984" y1="11.43" x2="25.4" y2="11.43" width="0.1524" layer="1"/>
+<wire x1="25.4" y1="11.3284" x2="25.4" y2="11.43" width="0.1524" layer="1"/>
 <wire x1="31.75" y1="26.67" x2="29.21" y2="26.67" width="0.1524" layer="1"/>
 <wire x1="28.0416" y1="20.8788" x2="28.0416" y2="19.9644" width="0.1524" layer="1"/>
@@
 <signal name="N$8">
 <contactref element="R2" pad="2"/>
-<contactref element="TP2" pad="TP"/>
-<wire x1="54.7116" y1="19.05" x2="54.7116" y2="21.4884" width="0.1524" layer="1"/>
-<wire x1="54.7116" y1="21.4884" x2="54.61" y2="21.59" width="0.1524" layer="1"/>
+<contactref element="CE" pad="TP"/>
+<wire x1="54.61" y1="19.05" x2="54.61" y2="21.59" width="0.1524" layer="1"/>
 <wire x1="54.7116" y1="19.05" x2="54.61" y2="19.05" width="0.1524" layer="1"/>
 </signal>
 <signal name="N$10">
 <contactref element="R4" pad="2"/>
-<contactref element="TP3" pad="TP"/>
-<wire x1="39.4716" y1="16.6116" x2="39.4716" y2="17.6784" width="0.1524" layer="1"/>
-<wire x1="39.4716" y1="17.6784" x2="39.37" y2="17.78" width="0.1524" layer="1"/>
-<wire x1="39.4716" y1="16.6116" x2="39.37" y2="16.51" width="0.1524" layer="1"/>
+<contactref element="CLK" pad="TP"/>
+<wire x1="39.37" y1="16.51" x2="39.37" y2="17.78" width="0.1524" layer="1"/>
 </signal>
 <signal name="N$11">
 <contactref element="R5" pad="2"/>
-<contactref element="TP4" pad="TP"/>
+<contactref element="DAT" pad="TP"/>
 <wire x1="36.8808" y1="46.9392" x2="36.8808" y2="45.72" width="0.1524" layer="1"/>
 <wire x1="36.8808" y1="45.72" x2="36.83" y2="45.72" width="0.1524" layer="1"/>
@@
 <signal name="N$17">
 <contactref element="R8" pad="2"/>
-<contactref element="TP5" pad="TP"/>
+<contactref element="MONO" pad="TP"/>
 <wire x1="54.7116" y1="29.2608" x2="54.7116" y2="31.6992" width="0.1524" layer="1"/>
 <wire x1="54.7116" y1="31.6992" x2="54.61" y2="31.75" width="0.1524" layer="1"/>
@@
 <contactref element="R11" pad="2"/>
 <contactref element="Q1" pad="C"/>
-<contactref element="TP6" pad="TP"/>
+<contactref element="TUNE" pad="TP"/>
 <wire x1="36.83" y1="49.53" x2="35.56" y2="49.53" width="0.1524" layer="1"/>
 <wire x1="36.8808" y1="49.53" x2="36.8808" y2="53.34" width="0.1524" layer="1"/>
@@
 <contactref element="Q2" pad="C"/>
 <contactref element="R13" pad="1"/>
-<contactref element="TP7" pad="TP"/>
+<contactref element="STEREO" pad="TP"/>
 <wire x1="48.3108" y1="52.1208" x2="45.72" y2="52.1208" width="0.1524" layer="1"/>
 <wire x1="49.53" y1="53.34" x2="48.3108" y2="52.1208" width="0.1524" layer="1"/>
